File: pcb/V2.3/recluse_fc.sch (KiCad schematic (older format))
At the start: 6 parts

Commit message: Ported V2.2 to KiCad
Parts:
- added C? (x2): 22uF, symbol Device:C_Small
- added C? (x4): 0.1uF, symbol Device:C_Small
- added C? (x2): 100nF, symbol Device:C_Small
- added C? (x2): 47uF, symbol Device:C_Small
- added C?: 2.2uF, symbol Device:C_Small
- added D? (x5): LTST-C190GKT, digikey-footprints:LED_0603, symbol dk_LED-Indication-Discrete:LTST-C190GKT
- added L? (x2): 10uH, symbol pspice:INDUCTOR
- added P?: USB_C_Plug_USB2.0, symbol Connector:USB_C_Plug_USB2.0
- added P?: VIN, symbol recluse:PAD
- added P?: GND, symbol recluse:PAD_GND
- added P?: S1, symbol recluse:PAD
- added P?: S2, symbol recluse:PAD
- added P?: S3, symbol recluse:PAD
- added P?: S4, symbol recluse:PAD
- added P? (x2): RX6, symbol recluse:PAD
- added Q?: AO3400A, Package_TO_SOT_SMD:SOT-23, symbol Transistor_FET:AO3400A
- added R? (x2): 1k, symbol Device:R_Small
- added R? (x2): 51k, symbol Device:R_Small
- added R? (x2): 41.2k, symbol Device:R_Small
- added R?: 6.68k, symbol Device:R_Small
- added R?: 4.64k, symbol Device:R_Small
- added R? (x2): 10k, symbol Device:R_Small
- added R? (x2): 5.1k, symbol Device:R_Small
- added R?: 47k, symbol Device:R_Small
- added R?: 220k, symbol Device:R_Small
- added R?: 620k, symbol Device:R_Small
- added R? (x2): 75k, symbol Device:R_Small
- added R?: 2.2k, symbol Device:R_Small
- added R?: 18k, symbol Device:R_Small
- added R?: 2k, symbol Device:R_Small
- added SW?: SW_Push_Dual_x2, symbol Switch:SW_Push_Dual_x2
- added U? (x2): MP4420GJ-P, Package_TO_SOT_SMD:TSOT-23-8, symbol recluse:MP4420GJ-P
- added U?: W25Q128JVS, Package_SO:SOIC-8_5.23x5.23mm_P1.27mm, symbol Memory_Flash:W25Q128JVS
- added U?: MPU-6000, Sensor_Motion:InvenSense_QFN-24_4x4mm_P0.5mm, symbol Sensor_Motion:MPU-6000
- added U?: USBLC6-4SC6, Package_TO_SOT_SMD:SOT-23-6, symbol Power_Protection:USBLC6-4SC6
- added X?: CSTNE8M00G520000R0, Crystal:Resonator_SMD_muRata_CSTxExxV-3Pin_3.0x1.1mm, symbol recluse:CSTNE8M00G520000R0
Connections:
- net +3V3: now also C?.2, D?.2, R?.1, R?.1, SW?.2 (D), U?.13 (VDD), U?.8 (VCC)
- net 9V_ENABLE: now also U?.6 (EN/SYNC)
- net ADC_CURR: now also P?.1
- net ADC_VBAT: now also R?.1, R?.2
- net BOOT: now also SW?.1 (C)
- net BUZZER: now also R?.1
- net CS_FLASH: now also U?.1 (~CS)
- net GND: now also C?.1, C?.1, C?.1, C?.2, C?.2, C?.2, C?.2, C?.2, C?.2, P?.1, P?.A1 (GND), P?.A12 (GND), P?.B1 (GND), P?.B12 (GND), P?.S1 (SHIELD), Q?.3 (D), R?.1, R?.1, R?.1, R?.1, R?.2, R?.2, R?.2, R?.2, R?.2, R?.2, U?.1 (CLKIN), U?.11 (FSYNC), U?.18 (GND), U?.2 (GND), U?.4 (GND), U?.4 (GND), U?.4 (GND), X?.2 (GND)
- net GYRO_CS: now also U?.8 (~CS)
- net GYRO_INT: now also U?.12 (INT)
- net GYRO_SCLK: now also U?.23 (SCL/SCLK)
- net LED0: now also D?.2
- net LED1: now also D?.2
- net OSC_IN: now also X?.1 (IN)
- net OSC_OUT: now also X?.3 (OUT)
- net S1: now also P?.1
- net S2: now also P?.1
- net S3: now also P?.1
- net S4: now also P?.1
- net SPI2_MISO: now also U?.2 (DO(IO1))
- net SPI2_MOSI: now also U?.5 (DI(IO0))
- net SPI2_SCK: now also U?.6 (CLK)
- net UART6_RX: now also P?.1
- net USB_D+: now also U?.4 (I/O3)
- net USB_D-: now also U?.6 (I/O4)
- net VBUS: now also P?.A4 (VBUS), P?.A9 (VBUS), P?.B4 (VBUS), P?.B9 (VBUS), U?.5 (VBUS); no longer D?.2
- net GYRO_SDI renamed GYRO_MOSI
- net GYRO_MOSI: now also U?.24 (SDA/MOSI)
- net GYRO_SDO renamed GYRO_MISO
- net GYRO_MISO: now also U?.9 (AD0/MISO)
- new net: C?.1, U?.2 (VCC), U?.~ (PG) (x2)
- new net: C?.1, R?.1 (x2)
- new net: R?.1, R?.2, R?.2 (x2)
- new net: R?.2, U?.3 (IO2)
- new net: R?.2, U?.7 (IO3)
- new net: C?.2, U?.10 (REGOUT)
- new net: C?.2, U?.20 (CPOUT)
- new net: P?.A5 (CC), R?.2
- new net: P?.B5 (VCONN), R?.2
- new net: D?.1, R?.1 (x5)
- new net: Q?.1 (G), R?.2
- new net +5V: C?.1, D?.2, D?.2, L?.2, R?.1
- new net +9V: C?.1, D?.2, L?.2, R?.1
- new net 5V_BST: R?.2, R?.2, U?.5 (BST)
- new net 5V_FB: R?.2, R?.2, U?.8 (FB)
- new net 5V_SW: C?.2, C?.2, L?.1, L?.1, U?.3 (SW)
- new net 9V_BST: U?.5 (BST)
- new net 9V_FB: U?.8 (FB)
- new net 9V_SW: U?.3 (SW)
- new net BUZZER-: Q?.2 (S)
- new net USB_CON_D+: P?.A6 (D+), U?.1 (I/O1)
- new net USB_CON_D-: P?.A7 (D-), U?.3 (I/O2)
- new net VIN: C?.1, C?.1, P?.1, R?.1, U?.2 (VCC), U?.2 (VCC)
- no-connect marks 13 -> 16
Other:
- note added: "3S-6S"
- note added: "5V DC-DC Buck Converter"
- note added: "9V DC-DC Buck Converter"
- note added: "According to datasheet\n"
- note added: "Dataflash (Blackbox)"
- note added: "ESC"
- note added: "MPU-6000"
- note added: "USB-C"
- moved on the sheet: C?, U?

Commit message: Completely ported EasyEda schematic to KiCad
Parts:
- added P1, P15, P16, P19, P31, P5, P9: GND, symbol recluse:PAD_GND
- added P10, P13, P2, P32, P6: 5V, symbol recluse:PAD
- added P11: TX5, symbol recluse:PAD
- added P12: RX5, symbol recluse:PAD
- added P14: LED, symbol recluse:PAD
- added P17: BUZZER-, symbol recluse:PAD
- added P18: BUZZER+, symbol recluse:PAD
- added P20: 9V, symbol recluse:PAD
- added P21: TX2, symbol recluse:PAD
- added P22: RX2, symbol recluse:PAD
- added P3: TX3, symbol recluse:PAD
- added P33: TX1, symbol recluse:PAD
- added P34: RX1, symbol recluse:PAD
- added P35: SCL, symbol recluse:PAD
- added P36: SDA, symbol recluse:PAD
- added P4: RX3, symbol recluse:PAD
- added P7: TX4, symbol recluse:PAD
- added P8: RX4, symbol recluse:PAD
- added R15, R16: 2.2k, symbol Device:R_Small
- gave numbers to parts that had none: 61
Connections:
- net +3V3: now also P18.1
- net +5V: now also P10.1, P13.1, P2.1, P32.1, P6.1
- net +9V: now also P20.1
- net BUZZER-: now also P17.1
- net GND: now also P1.1, P15.1, P16.1, P19.1, P31.1, P5.1, P9.1, R15.1, R16.1
- net I2C_SCL: now also P35.1, R16.2
- net LED_STRIP: now also P14.1
- net UART1_RX: now also P34.1
- net UART1_TX: now also P33.1
- net UART2_RX: now also P22.1
- net UART2_TX: now also P21.1
- net UART3_RX: now also P4.1
- net UART3_TX: now also P3.1
- net UART4_RX: now also P8.1
- net UART4_TX: now also P7.1
- net UART5_RX: now also P12.1
- net UART5_TX: now also P11.1
- new net I2C_SDA: P36.1, R15.2
Other:
- note added: "Breakouts\n"
- note added: "Buzzer\n"
- note added: "I2C Breakouts"
- note added: "Led Strip"
- note added: "UART 1"
- note added: "UART 2 (DJI)"
- note added: "UART 3"
- note added: "UART 4"
- note added: "UART 5"
- moved on the sheet: C12, C13, C14, C2, C3, C7, D1, D2, D3, D4, D5, D6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
